File: Lab4_board.kicad_pcb (KiCad board)
At the start: 2 copper layers, 66 x 66 mm, 21 parts, among them J1 PJ-102A, J2 Power Out, J3 Signals, U1 SN74LS138, U2 SN74LS138, U3 SN74LS04N, U4 SN74LS04N, U5 MIC29310-5.0WU-TR

Commit message: final version for 20882 matrix
Parts:
- added R9: 330, Resistors_SMD:R_0603, F.Cu at (124.9, 76.3)
- C1: value 0u1 -> 0u33
- C2: value 47u -> 0u1; footprint Capacitors_SMD:CP_Elec_5x5.8 -> Capacitors_SMD:C_0603
- U5: value MIC29310-5.0WU-TR -> uA7805; footprint TO_SOT_Packages_SMD:TO-263-3_TabPin4 -> Libraries:T0263-3
- moved C2 14.9 mm to (124.9, 74.5), turned to 180 degrees
- moved C1 7.86 mm to (121.4, 74.5), turned to 0 degrees
- moved U5 2.39 mm to (123.2, 60.2), turned to 0 degrees
Routing:
- net GND: track 9.15 -> 0.00 mm, vias 3 -> 8
- net Net-(C1-Pad1): track 15.0 -> 20.0 mm
- net VCC: track 82.9 -> 86.7 mm, vias 2 -> 1
